Commit message: made minor improvements

File: rover_project_ATT_OA/src/mobile_robot/model/rover.xacro (robot description, xacro)
@@ -1,406 +1,173 @@
-<?xml version = "1.0"?>
-<robot xmlns:xacro="http://www.ros.org/wiki/xacro" name= "rover">
-<xacro:property name = "base_link_x" value = "0.5"/>
-<xacro:property name = "base_link_y" value = "1.0"/>
-<xacro:property name = "base_link_z" value = "0.25"/>
-<xacro:property name = "wheel_link_radius" value = "0.15"/>
-<xacro:property name = "wheel_link_length" value = "0.05"/>
-<xacro:property name = "wheel_link_z" value = "-0.05"/>
-<xacro:property name = "chassis_length" value = "0.8"/>
-<xacro:property name = "chassis_width" value = "0.8"/>
-<xacro:property name = "chassis_height" value = "0.3"/>
-<xacro:property name = "wheel_radius" value = "0.20"/>
-<xacro:property name = "wheel_width" value = "0.10"/>
-<xacro:property name = "wheel_offset" value = "-0.10"/>
-<xacro:property name = "density" value = "2710.0"/>
-<xacro:property name = "pi_constant" value = "3.14159"/>
-<xacro:property name = "base_mass" value = "${2710.0*0.5*1.0*0.25}"/>
-<xacro:property name = "wheel_mass" value = "${2710.0*3.14159*0.15*0.15*0.05}"/>
-<xacro:property name = "Iz_wheel" value = "${0.5*9.5779*0.15*0.15}"/>
-<xacro:property name = "I_wheel" value = "${(1.0/12.0)*9.5779*(3.0*0.15*0.15+0.05*0.05)}"/>
-<xacro:macro name = "inertial_wheel">
-<inertial>
-<origin rpy = "0 0 0" xyz = "0 0 0"/>
-<mass value = "${9.5779}"/>
-<inertia ixx = "${I_wheel}" ixy = "0" ixz = "0" iyy = "${I_wheel}" iyz = "0" izz = "${Iz_wheel}" />
-</inertial>
+<?xml version="1.0"?>
+<robot xmlns:xacro="http://www.ros.org/wiki/xacro">
+<!-- ############################ PARAMETERS ############################# -->
+<xacro:property name="base_link_y" value="1.0"/>
+<xacro:property name="wheel_radius" value="0.15"/>
+<xacro:property name="wheel_width" value="0.05"/>
+<!-- ########################### PHYSICS PROPERTIES ###################### -->
+<gazebo reference="base_link">
+    <mu1>0.5</mu1>
+    <mu2>0.5</mu2>
+    <material>Gazebo/FlatBlack</material>
+    <kp>1e6</kp>
+    <kd>1e3</kd>
+</gazebo>
+<xacro:macro name="wheel_physics" params="link_name">
+    <gazebo reference="${link_name}">
+        <mu1>1.5</mu1>  <!-- Higher friction for wheels -->
+        <mu2>1.5</mu2>
+        <material>Gazebo/Rubber</material>
+        <kp>1e6</kp>
+        <kd>1e3</kd>
+    </gazebo>
 </xacro:macro>
-<xacro:include filename="$(find mobile_robot)/model/rover.gazebo"/>
-<material name = "black">
-    <color rgba = " 0 0 0 1"/>
-</material>
-<material name = "white">
-    <color rgba = " 1 1 1 1"/>
-</material>
-<material name = "green">
-    <color rgba = " 0 0.5 0 1"/>
-</material>
-<material name = "blue">
-    <color rgba = " 0 0 0.5 1"/>
-</material>
-<material name = "red">
-    <color rgba = " 0.5 0 0 1"/>
-</material>
-<link name = "dummy">
-</link>
-<joint name = "dummy_joint" type = "fixed">
-<parent link = "dummy"/>
-<child link = "base_link"/>
-</joint>
-    <link name = "base_link">
-        <visual>
-            <geometry>
-                <box size = "${0.5} ${1.0} ${0.25}"/>
-            </geometry>
-            <origin xyz = " 0 0 0.125" rpy = "0 0 0"/>
-            <material name = "black"/>
-        </visual>
-    <collision>
-            <geometry>
-                <box size = "${0.5} ${1.0} ${0.25}"/>
-            </geometry>
-            <origin xyz = " 0 0 0.125" rpy = "0 0 0"/>
-    </collision>
-    <inertial>
-        <origin xyz = " 0 0 0.125" rpy = "0 0 0"/>
-        <mass value= "${base_mass}"/>
-        <inertia ixx = "${(1.0/12.0)*base_mass*(1.0*1.0+0.25*0.25)}"
-        ixy = "0" ixz = "0"
-        iyy = "${(1.0/12.0)*base_mass*(0.5*0.5+0.25*0.25)}"
-        izz = "${(1.0/12.0)*base_mass*(1.0*1.0+0.5*0.5)}"
-        iyz = "0"/>
-    </inertial>
-    </link>
-<joint name = "left_front_wheel_joint" type = "continuous">
-    <parent link = "base_link"/>
-    <child link = "left_front_link"/>
-    <origin xyz = "0.275 ${-1.0/2.0-0.05/2.0} ${-0.05}" rpy = "0 0 0" />
-    <axis xyz ="1 0 0"/>
-    <limit effort = "1000" velocity = "1000"/>
-    <dynamics damping = "1.0" friction = "1.0"/>
-</joint>
-    <link name = "left_front_link">
-        <visual>
-            <geometry>
-                <cylinder radius = "${0.15}" length = "${0.05}"/>
-            </geometry>
-            <origin xyz = " 0 0 0" rpy = "0 1.570795 0"/>
-            <material name = "white"/>
-        </visual>
-    <collision>
-            <geometry>
-                 <cylinder radius = "${0.15}" length = "${0.05}"/>
-            </geometry>
-            <origin xyz = " 0 0 0" rpy = "0 1.570795 0"/>
-    </collision>
-<xacro:inertial_wheel/>
-    </link>
-<joint name = "right_front_wheel_joint" type = "continuous">
-    <parent link = "base_link"/>
-    <child link = "right_front_link"/>
-    <origin xyz = "-0.275 ${-1.0/2.0-0.05/2.0} ${-0.05}" rpy = "0 0 0" />
-    <axis xyz ="1 0 0"/>
-    <limit effort = "1000" velocity = "1000"/>
-    <dynamics damping = "1.0" friction = "1.0"/>
-</joint>
-    <link name = "right_front_link">
-        <visual>
-            <geometry>
-                <cylinder radius = "${0.15}" length = "${0.05}"/>
-            </geometry>
-            <origin xyz = " 0 0 0" rpy = "0 1.570795 0"/>
-            <material name = "white"/>
-        </visual>
-    <collision>
-            <geometry>
-                 <cylinder radius = "${0.15}" length = "${0.05}"/>
-            </geometry>
-            <origin xyz = " 0 0 0" rpy = "0 1.570795 0"/>
-    </collision>
-  <xacro:inertial_wheel/>
-    </link>
-<joint name = "left_back_wheel_joint" type = "continuous">
-    <parent link = "base_link"/>
-    <child link = "left_back_link"/>
-    <origin xyz = "0.275 ${1.0/2.0+0.05/2.0} ${-0.05}" rpy = "0 0 0" />
-    <axis xyz ="1 0 0"/>
-    <limit effort = "1000" velocity = "1000"/>
-    <dynamics damping = "1.0" friction = "1.0"/>
-</joint>
-    <link name = "left_back_link">
-        <visual>
-            <geometry>
-               <cylinder radius = "${0.15}" length = "${0.05}"/>
-            </geometry>
-            <origin xyz = " 0 0 0" rpy = "0 1.570795 0"/>
-            <material name = "white"/>
-        </visual>
-     <collision>
-            <geometry>
-                <cylinder radius = "${0.15}" length = "${0.05}"/>
-            </geometry>
-            <origin xyz = " 0 0 0" rpy = "0 1.570795 0"/>
-    </collision>
-    <xacro:inertial_wheel/>
-    </link>
-<joint name = "right_back_wheel_joint" type = "continuous">
-    <parent link = "base_link"/>
-    <child link = "right_back_link"/>
-    <origin xyz = "-0.275 ${1.0/2.0+0.05/2.0} ${-0.05}" rpy = "0 0 0" />
-    <axis xyz ="1 0 0"/>
-    <limit effort = "1000" velocity = "1000"/>
-    <dynamics damping = "1.0" friction = "1.0"/>
-</joint>
-    <link name = "right_back_link">
-        <visual>
-            <geometry>
-                 <cylinder radius = "${0.15}" length = "${0.05}"/>
-            </geometry>
-            <origin xyz = " 0 0 0" rpy = "0 1.570795 0"/>
-            <material name = "white"/>
-        </visual>
-     <collision>
-            <geometry>
-                <cylinder radius = "${0.15}" length = "${0.05}"/>
-            </geometry>
-            <origin xyz = " 0 0 0" rpy = "0 1.570795 0"/>
-    </collision>
-       <xacro:inertial_wheel/>
-    </link>
-<joint name="lidar_joint" type="fixed">
-    <parent link="base_link"/>
-    <child link="lidar_link"/>
-    <origin xyz="0 0 0.3" rpy="0 0 0"/>
-</joint>
- <link name="lidar_link">
-    <visual>
-      <geometry>
-        <cylinder radius="0.1" length="0.2"/>
-      </geometry>
-      <material name="blue"/>
-    </visual>
-    <collision>
-      <geometry>
-        <cylinder radius="0.05" length="0.1"/>
-      </geometry>
-    </collision>
-    <inertial>
-      <mass value="0.5"/>
-      <inertia ixx="0.01" ixy="0" ixz="0" iyy="0.01" iyz="0" izz="0.01"/>
-    </inertial>
-  </link>
-  <!-- Gazebo Plugin for Lidar -->
-  <gazebo reference="lidar_link">
-    <sensor name="lidar_sensor" type="ray">
-      <pose>0 0 0 0 0 0</pose>
-      <visualize>true</visualize>
-      <update_rate>10</update_rate>
-      <ray>
-        <scan>
-          <horizontal>
-            <samples>360</samples>
-            <resolution>1</resolution>
-            <min_angle>-3.14159</min_angle>
-            <max_angle>3.14159</max_angle>
-          </horizontal>
-        </scan>
-        <range>
-          <min>0.1</min>
-          <max>10.0</max>
-          <resolution>0.01</resolution>
-        </range>
-        <noise>
-          <type>gaussian</type>
-          <mean>0.0</mean>
-          <stddev>0.01</stddev>
-        </noise>
-      </ray>
-      <plugin name="lidar_plugin" filename="libgazebo_ros_ray_sensor.so">
-        <ros>
-          <namespace>lidar</namespace>
-          <remapping>~/out:=scan</remapping>
-        </ros>
-        <frame_name>lidar_link</frame_name>
-      </plugin>
+<xacro:wheel_physics link_name="left_front_link"/>
+<xacro:wheel_physics link_name="left_back_link"/>
+<xacro:wheel_physics link_name="right_front_link"/>
+<xacro:wheel_physics link_name="right_back_link"/>
+<!-- ######################## SENSOR CONFIGURATIONS ###################### -->
+<!-- Lidar Configuration -->
+<gazebo reference="lidar_link">
+    <material>Gazebo/Cobalt</material>
+    <sensor type="ray" name="main_lidar">
+        <pose>0 0 0 0 0 0</pose>
+        <visualize>true</visualize>
+        <update_rate>40</update_rate>
+        <ray>
+            <scan>
+                <horizontal>
+                    <samples>1080</samples>
+                    <resolution>0.33</resolution>
+                    <min_angle>${-pi}</min_angle>
+                    <max_angle>${pi}</max_angle>
+                </horizontal>
+                <vertical>
+                    <samples>16</samples>
+                    <resolution>0.01</resolution>
+                    <min_angle>-0.1</min_angle>
+                    <max_angle>0.1</max_angle>
+                </vertical>
+            </scan>
+            <range>
+                <min>0.25</min>
+                <max>30.0</max>
+                <resolution>0.03</resolution>
+            </range>
+            <noise>
+                <type>gaussian</type>
+                <mean>0.0</mean>
+                <stddev>0.0075</stddev>
+            </noise>
+        </ray>
+        <plugin name="lidar_controller" filename="libgazebo_ros_ray_sensor.so">
+            <topic_name>scan</topic_name>
+            <frame_name>lidar_link</frame_name>
+            <radiation_type>infrared</radiation_type>
+        </plugin>
     </sensor>
-  </gazebo>
-<gazebo>
-  <plugin name='skid_steer_drive' filename='libgazebo_ros_diff_drive.so'>
-    <ros>
-      <namespace></namespace>
-    </ros>
-    <num_wheel_pairs>2</num_wheel_pairs>
-    <wheel0>left_front_wheel_joint</wheel0>
-    <wheel1>right_front_wheel_joint</wheel1>
-    <wheel2>left_back_wheel_joint</wheel2>
-    <wheel3>right_back_wheel_joint</wheel3>
-    <wheel_separation>1.05</wheel_separation>
-    <wheel_diameter>0.15</wheel_diameter>
-    <max_wheel_torque>1000</max_wheel_torque>
-    <max_wheel_acceleration>5.0</max_wheel_acceleration>
-    <!-- Ensure the rover starts stationary -->
-    <init_velocity_x>0</init_velocity_x>
-    <init_velocity_y>0</init_velocity_y>
-    <init_velocity_yaw>0</init_velocity_yaw>
-  </plugin>
 </gazebo>
-<joint name="imu_joint" type="fixed">
-    <parent link="base_link"/>
-    <child link="imu_link"/>
-    <origin xyz="0 0 0.3" rpy="0 0 0"/>
-</joint>
-  <!-- IMU Link -->
-  <link name="imu_link">
-    <visual>
-      <geometry>
-        <cylinder radius="0.05" length="0.1"/>
-      </geometry>
-       <origin xyz="0 0 0" rpy="0 0 0"/>
-      <material name="black">
-        <color rgba="0 1 0 1"/>
-      </material>
-    </visual>
-    <collision>
-      <geometry>
-        <cylinder radius="0.05" length="0.04"/>
-      </geometry>
-    </collision>
-</link>
-  <gazebo reference="imu_link">
+<!-- IMU Configuration -->
+<gazebo reference="imu_link">
     <sensor name="imu_sensor" type="imu">
-      <always_on>true</always_on>
-      <update_rate>10.0</update_rate>
-      <plugin name="imu_controller" filename="libgazebo_ros_imu_sensor.so">
-        <ros>
-          <remapping>imu_controller/out:=imu</remapping>
-        </ros>
-        <frame_name>imu_link</frame_name>
-      </plugin>
+        <always_on>true</always_on>
+        <update_rate>400</update_rate>
+        <imu>
+            <noise>
+                <type>gaussian</type>
+                <rate>
+                    <mean>0.0</mean>
+                    <stddev>0.00017</stddev>
+                    <bias_mean>0.0001</bias_mean>
+                    <bias_stddev>0.0001</bias_stddev>
+                </rate>
+                <accel>
+                    <mean>0.0</mean>
+                    <stddev>0.0028</stddev>
+                    <bias_mean>0.1</bias_mean>
+                    <bias_stddev>0.001</bias_stddev>
+                </accel>
+            </noise>
+        </imu>
+        <plugin filename="libgazebo_ros_imu_sensor.so" name="imu_plugin">
+            <topic_name>imu/data</topic_name>
+            <frame_name>imu_link</frame_name>
+            <initial_orientation_as_reference>false</initial_orientation_as_reference>
+        </plugin>
     </sensor>
-    <material>Gazebo/Grey</material>
-  </gazebo>
-    <!-- GPS Sensor -->
-  <link name="gps_link">
-    <visual>
-      <geometry>
-        <cylinder radius="0.05" length="0.3"/>
-      </geometry>
-      <origin xyz="0 0 0" rpy="0 0 0"/>
-      <material name="black">
-        <color rgba="0 1 0 1"/>
-      </material>
-    </visual>
-    <collision>
-      <geometry>
-        <cylinder radius="0.05" length="0.04"/>
-      </geometry>
-    </collision>
-    </link>
+</gazebo>
+<!-- GPS Configuration -->
 <gazebo reference="gps_link">
     <sensor name="gps_sensor" type="gps">
         <always_on>true</always_on>
-        <update_rate>1.0</update_rate>
-        <plugin name="gps_controller" filename="libgazebo_ros_gps_sensor.so">
-            <ros>
-                <remapping>gps_controller/out:=gps</remapping>
-            </ros>
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